Commit message: Create gpu to enable/disable GPU processing

File: ca_description/urdf/roomblock.xacro (robot description, xacro)
@@ -8,5 +8,5 @@
   <xacro:include filename="$(find ca_description)/urdf/sensors/laser_sensor.xacro"/>
   <xacro:include filename="$(find ca_description)/urdf/sensors/camera_sensor.xacro"/>
-  <xacro:macro name="roomblock" params="parent visualize:=false">
+  <xacro:macro name="roomblock" params="parent visualize:=false gpu:=false">
     <xacro:property name="z" value="0.07"/>
     <xacro:property name="roomblock_link" value="block_link"/>
@@ -35,5 +35,5 @@
       </xacro:inertial_cuboid_with_pose>
     </link>
-    <xacro:laser_sensor parent="${roomblock_link}" visualize="$(arg visualize)"/>
+    <xacro:laser_sensor parent="${roomblock_link}" visualize="${visualize}" gpu="${gpu}"/>
     <xacro:camera_sensor parent="${roomblock_link}"/>
     <xacro:roomblock_gazebo link_name="${roomblock_link}"/>
