Commit message: Add GPU flag

File: ca_description/urdf/create_base.xacro (robot description, xacro)
@@ -1,5 +1,5 @@
 <?xml version="1.0" ?>
 <robot xmlns:xacro="http://ros.org/wiki/xacro">
-  <xacro:macro name="create_base" params="wheel_separation wheel_radius wheel_width base_diameter *mesh visualize:=false">
+  <xacro:macro name="create_base" params="wheel_separation wheel_radius wheel_width base_diameter *mesh visualize:=false gpu:=false">
     <xacro:include filename="$(find ca_description)/urdf/create_base_gazebo.xacro"/>
     <xacro:include filename="$(find ca_description)/urdf/create_caster_wheel.xacro"/>
@@ -36,6 +36,6 @@
       </collision>
     </link>
-    <xacro:wall_sensor visualize="${visualize}"/>
-    <xacro:cliff_sensors visualize="${visualize}"/>
+    <xacro:wall_sensor visualize="${visualize}" gpu="${gpu}"/>
+    <xacro:cliff_sensors visualize="${visualize}" gpu="${gpu}"/>
     <xacro:imu_sensor name="imu">
       <origin xyz="0 -0.04 0.13" rpy="0 0 0"/>

Commit message: Add wirtual wall
Signed-off-by: ivan <ivanpauno@gmail.com>

File: ca_description/urdf/create_base.xacro (robot description, xacro)
@@ -8,4 +8,5 @@
     <xacro:include filename="$(find ca_description)/urdf/sensors/wall_sensor.xacro"/>
     <xacro:include filename="$(find ca_description)/urdf/sensors/cliff_sensors.xacro"/>
+    <xacro:include filename="$(find ca_description)/urdf/sensors/virtual_wall_sensor.xacro"/>
     <xacro:property name="base_link_offset_z" value="0.0308"/>
     <xacro:property name="base_offset_z" value="0.017"/>
@@ -41,4 +42,7 @@
       <origin xyz="0 -0.04 0.13" rpy="0 0 0"/>
     </xacro:imu_sensor>
+    <xacro:virtual_wall_sensor name="virtual_wall_sensor" fov="0.1">
+      <origin xyz="0.145 0 ${base_link_offset_z}" rpy="0 0 0"/>
+    </xacro:virtual_wall_sensor>
     <xacro:create_wheel prefix="left" y_offset="${wheel_separation / 2}" wheel_radius="${wheel_radius}" wheel_width="${wheel_width}"/>
     <xacro:create_wheel prefix="right" y_offset="${wheel_separation / -2}" wheel_radius="${wheel_radius}" wheel_width="${wheel_width}"/>

Commit message: Corrections
Signed-off-by: ivanpauno <ivanpauno@ekumenlabs.com>

File: ca_description/urdf/create_base.xacro (robot description, xacro)
@@ -43,5 +43,5 @@
     </xacro:imu_sensor>
     <xacro:virtual_wall_sensor name="virtual_wall_sensor" fov="0.1">
-      <origin xyz="0.145 0 ${base_link_offset_z}" rpy="0 0 0"/>
+      <origin xyz="-0.145 0 ${base_link_offset_z}" rpy="0 0 0"/>
     </xacro:virtual_wall_sensor>
     <xacro:create_wheel prefix="left" y_offset="${wheel_separation / 2}" wheel_radius="${wheel_radius}" wheel_width="${wheel_width}"/>

Commit message: Address Emi's comments
Signed-off-by: ivanpauno <ivanpauno@ekumenlabs.com>

File: ca_description/urdf/create_base.xacro (robot description, xacro)
@@ -8,5 +8,5 @@
     <xacro:include filename="$(find ca_description)/urdf/sensors/wall_sensor.xacro"/>
     <xacro:include filename="$(find ca_description)/urdf/sensors/cliff_sensors.xacro"/>
-    <xacro:include filename="$(find ca_description)/urdf/sensors/virtual_wall_sensor.xacro"/>
+    <xacro:include filename="$(find ca_description)/urdf/sensors/omni_sensor.xacro"/>
     <xacro:property name="base_link_offset_z" value="0.0308"/>
     <xacro:property name="base_offset_z" value="0.017"/>
@@ -42,7 +42,7 @@
       <origin xyz="0 -0.04 0.13" rpy="0 0 0"/>
     </xacro:imu_sensor>
-    <xacro:virtual_wall_sensor name="virtual_wall_sensor" fov="0.1">
+    <xacro:omni_sensor name="omni_sensor" diameter="0.1">
       <origin xyz="-0.145 0 ${base_link_offset_z}" rpy="0 0 0"/>
-    </xacro:virtual_wall_sensor>
+    </xacro:omni_sensor>
     <xacro:create_wheel prefix="left" y_offset="${wheel_separation / 2}" wheel_radius="${wheel_radius}" wheel_width="${wheel_width}"/>
     <xacro:create_wheel prefix="right" y_offset="${wheel_separation / -2}" wheel_radius="${wheel_radius}" wheel_width="${wheel_width}"/>

File: ca_description/urdf/sensors/omni_sensor.xacro (robot description, xacro)
@@ -1,7 +1,7 @@
 <?xml version="1.0" ?>
 <robot xmlns:xacro="http://ros.org/wiki/xacro">
-<xacro:macro name="virtual_wall_sensor" params="name fov *origin">
+<xacro:macro name="omni_sensor" params="name diameter *origin">
   <xacro:include filename="$(find ca_description)/urdf/common_properties.xacro"/>
-  <xacro:include filename="$(find ca_description)/urdf/sensors/virtual_wall_sensor_gazebo.xacro"/>
+  <xacro:include filename="$(find ca_description)/urdf/sensors/omni_sensor_gazebo.xacro"/>
   <xacro:property name="parent_link" value="base_link"/>
   <xacro:property name="link_name" value="${name}_link"/>
@@ -14,5 +14,5 @@
     <xacro:dummy_inertia/>
   </link>
-  <xacro:virtual_wall_sensor_gazebo name="${name}" fov="${fov}"/>
+  <xacro:omni_sensor_gazebo name="${name}" diameter="${diameter}"/>
 </xacro:macro>
 </robot>

Commit message: Address newer comments
Signed-off-by: ivanpauno <ivanpauno@ekumenlabs.com>

File: ca_description/urdf/create_base.xacro (robot description, xacro)
@@ -43,5 +43,5 @@
     </xacro:imu_sensor>
     <xacro:omni_sensor name="omni_sensor" diameter="0.1">
-      <origin xyz="-0.145 0 ${base_link_offset_z}" rpy="0 0 0"/>
+      <origin xyz="0.145 0 ${base_link_offset_z}" rpy="0 0 0"/>
     </xacro:omni_sensor>
     <xacro:create_wheel prefix="left" y_offset="${wheel_separation / 2}" wheel_radius="${wheel_radius}" wheel_width="${wheel_width}"/>

File: ca_description/urdf/sensors/omni_sensor.xacro (robot description, xacro)
@@ -6,5 +6,5 @@
   <xacro:property name="parent_link" value="base_link"/>
   <xacro:property name="link_name" value="${name}_link"/>
-  <joint name="${name}_joint" type="continuous">
+  <joint name="${name}_joint" type="fixed">
     <xacro:insert_block name="origin" />
     <parent link="${parent_link}" />

Commit message: Added *origin block

File: ca_description/urdf/create_base.xacro (robot description, xacro)
@@ -45,6 +45,10 @@
     <xacro:create_wheel prefix="right" y_offset="${wheel_separation / -2}" wheel_radius="${wheel_radius}" wheel_width="${wheel_width}"/>
     <xacro:caster_wheel/>
-    <xacro:color_sensor parent="base_link" reflect="1" prefix="right"/>
-    <xacro:color_sensor parent="base_link" reflect="-1" prefix="left"/>
+    <xacro:color_sensor parent="base_link" reflect="1" prefix="right">
+      <origin xyz="0.05 0 0" rpy="${-pi/2} 0 ${-pi/2}" />
+    </xacro:color_sensor>
+    <xacro:color_sensor parent="base_link" reflect="-1" prefix="left">
+      <origin xyz="0.05 0 0" rpy="${-pi/2} 0 ${-pi/2}" />
+    </xacro:color_sensor>
     <!-- Simulation sensors -->
     <xacro:sim_create_base/>

File: ca_description/urdf/sensors/ramiro_color_sensor.xacro (robot description, xacro)
@@ -3,5 +3,5 @@
   <xacro:include filename="$(find ca_description)/urdf/sensors/laser_sensor_gazebo.xacro"/>
   <xacro:include filename="$(find ca_description)/urdf/common_properties.xacro"/>
-  <xacro:macro name="color_sensor" params="prefix reflect parent visualize:=false">
+  <xacro:macro name="color_sensor" params="prefix reflect parent visualize:=false *origin">
     <xacro:property name="parent_link" value="${parent}"/>
     <xacro:property name="color_sensor_len" value="0.05"/>
@@ -19,5 +19,5 @@
     </joint>
     <joint name="${prefix}_color_optical_joint" type="fixed">
-      <origin xyz="0.05 0 0" rpy="${-pi/2} 0 ${-pi/2}" />
+      <xacro:insert_block name="origin" />
       <parent link="${prefix}_color_sensor" />
       <child link="${prefix}_color_optical_frame"/>

Commit message: Removed `reflect` parameter on the `color_sensor` macro

File: ca_description/urdf/create_base.xacro (robot description, xacro)
@@ -45,8 +45,10 @@
     <xacro:create_wheel prefix="right" y_offset="${wheel_separation / -2}" wheel_radius="${wheel_radius}" wheel_width="${wheel_width}"/>
     <xacro:caster_wheel/>
-    <xacro:color_sensor parent="base_link" reflect="1" prefix="right">
+    <xacro:color_sensor parent="base_link" prefix="right">
+      <origin xyz="0.18 .08 0.1"  rpy="0 ${0.7*(pi/2)} 1"/>
       <origin xyz="0.05 0 0" rpy="${-pi/2} 0 ${-pi/2}" />
     </xacro:color_sensor>
-    <xacro:color_sensor parent="base_link" reflect="-1" prefix="left">
+    <xacro:color_sensor parent="base_link" prefix="left">
+      <origin xyz="0.18 -.08 0.1"  rpy="0 ${0.7*(pi/2)} -1"/>
       <origin xyz="0.05 0 0" rpy="${-pi/2} 0 ${-pi/2}" />
     </xacro:color_sensor>

File: ca_description/urdf/sensors/color_sensor.xacro (robot description, xacro)
@@ -3,5 +3,5 @@
   <xacro:include filename="$(find ca_description)/urdf/sensors/laser_sensor_gazebo.xacro"/>
   <xacro:include filename="$(find ca_description)/urdf/common_properties.xacro"/>
-  <xacro:macro name="color_sensor" params="prefix reflect parent visualize:=false *origin">
+  <xacro:macro name="color_sensor" params="prefix parent visualize:=false *origin1 **origin2">
     <xacro:property name="parent_link" value="${parent}"/>
     <xacro:property name="color_sensor_len" value="0.05"/>
@@ -16,8 +16,8 @@
         <parent link="${parent_link}"/>
         <child link="${prefix}_color_sensor"/>
-        <origin xyz="0.18 ${reflect*(.08)} 0.1"  rpy="0 ${0.7*(pi/2)} ${reflect}"/>
+        <xacro:insert_block name="origin1" />
     </joint>
     <joint name="${prefix}_color_optical_joint" type="fixed">
-      <xacro:insert_block name="origin" />
+      <xacro:insert_block name="origin2" />
       <parent link="${prefix}_color_sensor" />
       <child link="${prefix}_color_optical_frame"/>

Commit message: Add color sensor
Applied changes requested

Adressed the issues commented

Fixed type

Update sensor model

Added camera mesh

File: ca_description/urdf/create_base.xacro (robot description, xacro)
@@ -8,4 +8,5 @@
     <xacro:include filename="$(find ca_description)/urdf/sensors/wall_sensor.xacro"/>
     <xacro:include filename="$(find ca_description)/urdf/sensors/cliff_sensors.xacro"/>
+    <xacro:include filename="$(find ca_description)/urdf/color_sensor.xacro"/>
     <xacro:property name="base_link_offset_z" value="0.0308"/>
     <xacro:property name="base_offset_z" value="0.017"/>
@@ -36,4 +37,13 @@
       </collision>
     </link>
+    <xacro:property name="diameter" value="0.3485"/>
+    <xacro:property name="size_z" value="0.1"/>
+    <!-- Introducing color sensors in each side -->
+    <xacro:color_sensor prefix="left" parent="base_link" color="yellow">
+      <origin xyz="${diameter/2 * 0.5 + 0.03} ${diameter/2 * 0.84 } ${size_z}" rpy="0 ${pi/2} 0" />
+    </xacro:color_sensor>
+    <xacro:color_sensor prefix="right" parent="base_link" color="white">
+      <origin xyz="${diameter/2 * 0.5 + 0.05} ${-(diameter/2 * 0.63 )} ${size_z}" rpy="0 ${pi/2} 0"/>
+    </xacro:color_sensor>
     <xacro:wall_sensor visualize="${visualize}"/>
     <xacro:cliff_sensors visualize="${visualize}"/>

Commit message: Add color sensor
Applied changes requested

First draft

Changed code and added path node

Adressed some issues

File: ca_description/urdf/create_base.xacro (robot description, xacro)
@@ -8,4 +8,5 @@
     <xacro:include filename="$(find ca_description)/urdf/sensors/wall_sensor.xacro"/>
     <xacro:include filename="$(find ca_description)/urdf/sensors/cliff_sensors.xacro"/>
+    <xacro:include filename="$(find ca_description)/urdf/color_sensor.xacro"/>
     <xacro:property name="base_link_offset_z" value="0.0308"/>
     <xacro:property name="base_offset_z" value="0.017"/>
@@ -36,4 +37,8 @@
       </collision>
     </link>
+    <xacro:property name="diameter" value="0.3485"/>
+    <!-- Introducing color sensors in each side -->
+    <xacro:color_sensor prefix="left" side="${diameter}"/>
+    <xacro:color_sensor prefix="right" side="${-diameter}"/>
     <xacro:wall_sensor visualize="${visualize}"/>
     <xacro:cliff_sensors visualize="${visualize}"/>

Commit message: Moving origin block to the macro

File: ca_description/urdf/create_base.xacro (robot description, xacro)
@@ -45,11 +45,9 @@
     <xacro:create_wheel prefix="right" y_offset="${wheel_separation / -2}" wheel_radius="${wheel_radius}" wheel_width="${wheel_width}"/>
     <xacro:caster_wheel/>
-    <xacro:color_sensor parent="base_link" prefix="right">
+    <xacro:color_sensor parent="base_link" name_prefix="right">
       <origin xyz="0.18 .08 0.1"  rpy="0 ${0.7*(pi/2)} 1"/>
-      <origin xyz="0.05 0 0" rpy="${-pi/2} 0 ${-pi/2}" />
     </xacro:color_sensor>
-    <xacro:color_sensor parent="base_link" prefix="left">
+    <xacro:color_sensor parent="base_link" name_prefix="left">
       <origin xyz="0.18 -.08 0.1"  rpy="0 ${0.7*(pi/2)} -1"/>
-      <origin xyz="0.05 0 0" rpy="${-pi/2} 0 ${-pi/2}" />
     </xacro:color_sensor>
     <!-- Simulation sensors -->

File: ca_description/urdf/sensors/color_sensor.xacro (robot description, xacro)
@@ -2,7 +2,7 @@
 <robot xmlns:xacro="http://ros.org/wiki/xacro">
   <xacro:include filename="$(find ca_description)/urdf/common_properties.xacro"/>
-  <xacro:macro name="color_sensor" params="prefix parent visualize:=false *origin1 **origin2">
+  <xacro:macro name="color_sensor" params="name_prefix parent visualize:=false *origin">
     <xacro:property name="parent_link" value="${parent}"/>
-    <link name="${prefix}_color_sensor">
+    <link name="${name_prefix}_color_sensor">
         <visual>
             <geometry>
@@ -11,15 +11,15 @@
         </visual>
     </link>
-    <joint name="base_to_${prefix}_color_sensor" type="fixed">
+    <joint name="base_to_${name_prefix}_color_sensor" type="fixed">
         <parent link="${parent_link}"/>
-        <child link="${prefix}_color_sensor"/>
-        <xacro:insert_block name="origin1" />
+        <child link="${name_prefix}_color_sensor"/>
+        <xacro:insert_block name="origin" />
     </joint>
-    <joint name="${prefix}_color_optical_joint" type="fixed">
-      <xacro:insert_block name="origin2" />
-      <parent link="${prefix}_color_sensor" />
-      <child link="${prefix}_color_optical_frame"/>
+    <joint name="${name_prefix}_color_optical_joint" type="fixed">
+        <origin xyz="0.05 0 0" rpy="${-pi/2} 0 ${-pi/2}" />
+      <parent link="${name_prefix}_color_sensor" />
+      <child link="${name_prefix}_color_optical_frame"/>
     </joint>
-    <link name="${prefix}_color_optical_frame"/>
+    <link name="${name_prefix}_color_optical_frame"/>
  </xacro:macro>
 </robot>

Commit message: Adding new world
Added world and models

Big changes,added launch file, apriltag on create robot, erased to cameras, cleaned the world file

Changed the apriltags and camera plugin

fixup! Adding new world

Change apriltags for improve the visualization

Added in launch file apriltag and tf_state nodes

File: ca_description/urdf/create_base.xacro (robot description, xacro)
@@ -8,4 +8,5 @@
     <xacro:include filename="$(find ca_description)/urdf/sensors/wall_sensor.xacro"/>
     <xacro:include filename="$(find ca_description)/urdf/sensors/cliff_sensors.xacro"/>
+    <xacro:include filename="$(find ca_description)/urdf/create_apriltag.xacro"/>
     <xacro:property name="base_link_offset_z" value="0.0308"/>
     <xacro:property name="base_offset_z" value="0.017"/>
@@ -41,4 +42,7 @@
       <origin xyz="0 -0.04 0.13" rpy="0 0 0"/>
     </xacro:imu_sensor>
+    <xacro:create_apriltag parent="base_link">
+      <origin xyz="0 0 0.25"  rpy="0 0 0"/>
+    </xacro:create_apriltag>
     <xacro:create_wheel prefix="left" y_offset="${wheel_separation / 2}" wheel_radius="${wheel_radius}" wheel_width="${wheel_width}"/>
     <xacro:create_wheel prefix="right" y_offset="${wheel_separation / -2}" wheel_radius="${wheel_radius}" wheel_width="${wheel_width}"/>

Commit message: Added color sensor plugin

File: ca_description/urdf/create_base.xacro (robot description, xacro)
@@ -45,8 +45,8 @@
     <xacro:create_wheel prefix="right" y_offset="${wheel_separation / -2}" wheel_radius="${wheel_radius}" wheel_width="${wheel_width}"/>
     <xacro:caster_wheel/>
-    <xacro:color_sensor parent="base_link" name_prefix="right">
+    <xacro:color_sensor parent="base_link" name_prefix="left" color="yellow">
       <origin xyz="0.18 .08 0.1"  rpy="0 ${0.7*(pi/2)} 1"/>
     </xacro:color_sensor>
-    <xacro:color_sensor parent="base_link" name_prefix="left">
+    <xacro:color_sensor parent="base_link" name_prefix="right" color="white">
       <origin xyz="0.18 -.08 0.1"  rpy="0 ${0.7*(pi/2)} -1"/>
     </xacro:color_sensor>

File: ca_description/urdf/sensors/color_sensor.xacro (robot description, xacro)
@@ -2,5 +2,5 @@
 <robot xmlns:xacro="http://ros.org/wiki/xacro">
   <xacro:include filename="$(find ca_description)/urdf/common_properties.xacro"/>
-  <xacro:macro name="color_sensor" params="name_prefix parent visualize:=false *origin">
+  <xacro:macro name="color_sensor" params="name_prefix color parent visualize:=false *origin">
     <xacro:property name="parent_link" value="${parent}"/>
     <link name="${name_prefix}_color_sensor">
@@ -22,4 +22,40 @@
     </joint>
     <link name="${name_prefix}_color_optical_frame"/>
+    <gazebo reference="${name_prefix}_color_sensor">
+        <sensor name='camera' type='camera'>
+        <camera name='__default__'>
+         <horizontal_fov>0.3</horizontal_fov>
+         <image>
+           <width>120</width>
+           <height>120</height>
+         </image>
+         <clip>
+           <near>0.1</near>
+           <far>100</far>
+         </clip>
+       </camera>
+       <plugin name="gazebo_light_sensor_plugin" filename="libgazebo_color_plugin.so">
+         <publishTopic>${name_prefix}_color_sensor</publishTopic>
+         <sensorColor>${color}</sensorColor>
+         <cameraName>${name_prefix}</cameraName>
+         <always_on>true</always_on>
+         <update_rate>10</update_rate>
+         <imageTopicName>rgb/image_raw</imageTopicName>
+         <depthImageTopicName>depth/image_raw</depthImageTopicName>
+         <pointCloudTopicName>depth/points</pointCloudTopicName>
+         <cameraInfoTopicName>rgb/camera_info</cameraInfoTopicName>
+         <depthImageCameraInfoTopicName>depth/camera_info</depthImageCameraInfoTopicName>
+         <frameName>camera_depth_optical_frame</frameName>
+         <baseline>0.1</baseline>
+         <distortion_k1>0.0</distortion_k1>
+         <distortion_k2>0.0</distortion_k2>
+         <distortion_k3>0.0</distortion_k3>
+         <distortion_t1>0.0</distortion_t1>
+         <distortion_t2>0.0</distortion_t2>
+         <pointCloudCutoff>0.4</pointCloudCutoff>
+         <robotNamespace>/</robotNamespace>
+        </plugin>
+      </sensor>
+    </gazebo>
  </xacro:macro>
 </robot>

Commit message: Modified sensors positioning for better viewing of the lines

File: ca_description/urdf/create_base.xacro (robot description, xacro)
@@ -46,8 +46,8 @@
     <xacro:caster_wheel/>
     <xacro:color_sensor parent="base_link" name_prefix="left" color="yellow">
-      <origin xyz="0.18 .08 0.1"  rpy="0 ${0.7*(pi/2)} 1"/>
+      <origin xyz="0.18 .11 0.15"  rpy="0 ${(pi/2)} 0"/>
     </xacro:color_sensor>
     <xacro:color_sensor parent="base_link" name_prefix="right" color="white">
-      <origin xyz="0.18 -.08 0.1"  rpy="0 ${0.7*(pi/2)} -1"/>
+      <origin xyz="0.18 -.11 0.15"  rpy="0 ${(pi/2)} 0"/>
     </xacro:color_sensor>
     <!-- Simulation sensors -->

File: ca_description/urdf/sensors/color_sensor.xacro (robot description, xacro)
@@ -27,10 +27,10 @@
          <horizontal_fov>0.3</horizontal_fov>
          <image>
-           <width>120</width>
-           <height>120</height>
+           <width>200</width>
+           <height>200</height>
          </image>
          <clip>
            <near>0.1</near>
-           <far>100</far>
+           <far>10</far>
          </clip>
        </camera>
@@ -40,5 +40,5 @@
          <cameraName>${name_prefix}</cameraName>
          <always_on>true</always_on>
-         <update_rate>10</update_rate>
+         <update_rate>60</update_rate>
          <imageTopicName>rgb/image_raw</imageTopicName>
          <depthImageTopicName>depth/image_raw</depthImageTopicName>
