Commit message: Added visuals for sensors
Also added the optical frame link, with proper axis

File: ca_description/urdf/sensors/ramiro_color_sensor.xacro (robot description, xacro)
@@ -30,11 +30,4 @@
   <xacro:macro name="color_sensor" params="prefix reflect parent visualize:=false">
     <xacro:property name="parent_link" value="${parent}"/>
-    <xacro:property name="color_link" value="color_link"/>
-    <xacro:property name="x" value="0.0"/>
-    <xacro:property name="y" value="0.0"/>
-    <xacro:property name="z" value="0.3"/>
-    <xacro:property name="R" value="0.0"/>
-    <xacro:property name="P" value="0.0"/>
-    <xacro:property name="Y" value="0.45"/>
     <xacro:property name="color_sensor_len" value="0.05"/>
     <link name="${prefix}_color_sensor">
@@ -43,7 +36,8 @@
                 <box size="${color_sensor_len} 0.02 0.02"/>
             </geometry>
-            <origin xyz="0 0 -${color_sensor_len/2}"/>
+            <origin xyz="-${color_sensor_len/2} 0 0"/>
             <material name="white"/>
         </visual>
+    </link>
      <!--   <collision>
             <geometry>
@@ -54,10 +48,15 @@
         <xacro:default_inertial mass="10"/>
          -->
-    </link>
     <joint name="base_to_${prefix}_color_sensor" type="fixed">
         <parent link="${parent_link}"/>
         <child link="${prefix}_color_sensor"/>
-        <origin xyz="0.18 ${reflect*(.08)} 0.15" rpy="0 ${0.7*(pi/2)} ${reflect}"/>
+        <origin xyz="0.18 ${reflect*(.08)} 0.1"  rpy="0 ${0.7*(pi/2)} ${reflect}"/>
     </joint>
+    <joint name="${prefix}_color_optical_joint" type="fixed">
+      <origin xyz="0 0 0" rpy="${-pi/2} 0 ${-pi/2}" />
+      <parent link="${prefix}_color_sensor" />
+      <child link="${prefix}_color_optical_frame"/>
+    </joint>
+    <link name="${prefix}_color_optical_frame"/>
  </xacro:macro>
 </robot>

Commit message: Added mesh for visuals

File: ca_description/urdf/sensors/ramiro_color_sensor.xacro (robot description, xacro)
@@ -34,8 +34,7 @@
         <visual>
             <geometry>
-                <box size="${color_sensor_len} 0.02 0.02"/>
+                <mesh filename="package://ca_description/meshes/last_lens.stl" scale="0.0005 0.0005 0.0005" />
             </geometry>
-            <origin xyz="-${color_sensor_len/2} 0 0"/>
-            <material name="white"/>
+            <origin xyz="0 0 0" rpy="0 ${pi/2} 0"/>
         </visual>
     </link>
@@ -54,5 +53,5 @@
     </joint>
     <joint name="${prefix}_color_optical_joint" type="fixed">
-      <origin xyz="0 0 0" rpy="${-pi/2} 0 ${-pi/2}" />
+      <origin xyz="0.05 0 0" rpy="${-pi/2} 0 ${-pi/2}" />
       <parent link="${prefix}_color_sensor" />
       <child link="${prefix}_color_optical_frame"/>

Commit message: Reworked mesh with a visual tool
Deleted unused meshes

File: ca_description/urdf/sensors/ramiro_color_sensor.xacro (robot description, xacro)
@@ -3,29 +3,4 @@
   <xacro:include filename="$(find ca_description)/urdf/sensors/laser_sensor_gazebo.xacro"/>
   <xacro:include filename="$(find ca_description)/urdf/common_properties.xacro"/>
-<!--
-  <xacro:macro name="color_sensor" params="parent visualize:=false">
-    <xacro:property name="parent_link" value="${parent}"/>
-    <xacro:property name="color_link" value="color_link"/>
-    <xacro:property name="x" value="0.0"/>
-    <xacro:property name="y" value="0.0"/>
-    <xacro:property name="z" value="0.1308"/>
-    <xacro:property name="R" value="0.0"/>
-    <xacro:property name="P" value="0.0"/>
-    <xacro:property name="Y" value="${pi}"/>
-    <joint name="color_joint" type="fixed">
-      <origin xyz="${x} ${y} ${z}" rpy="${R} ${P} ${Y}" />
-      <parent link="${parent_link}" />
-      <child link="${color_link}" />
-    </joint>
-    <link name="${color_link}">
-       <visual>
-        <origin xyz="0 0 0" rpy="0 0 0" />
-        <geometry>
-         <box size="0.06 0.02 0.02" />
-        </geometry>
-       </visual>
-   </link>
-  </xacro:macro>
-  -->
   <xacro:macro name="color_sensor" params="prefix reflect parent visualize:=false">
     <xacro:property name="parent_link" value="${parent}"/>
@@ -34,17 +9,8 @@
         <visual>
             <geometry>
-                <mesh filename="package://ca_description/meshes/last_lens.stl" scale="0.0005 0.0005 0.0005" />
+                <mesh filename="package://ca_description/meshes/scaled_lens.stl"/>
             </geometry>
-            <origin xyz="0 0 0" rpy="0 ${pi/2} 0"/>
         </visual>
     </link>
-     <!--   <collision>
-            <geometry>
-                <box size="${color_sensor_len} 0.1 0.2"/>
-            </geometry>
-            <origin xyz="0 0 -${color_sensor_len/2}" rpy="0 ${pi/2} 0"/>
-        </collision>
-        <xacro:default_inertial mass="10"/>
-         -->
     <joint name="base_to_${prefix}_color_sensor" type="fixed">
         <parent link="${parent_link}"/>
