Commit message: Deleted unused parameter

File: ca_description/urdf/sensors/color_sensor.xacro (robot description, xacro)
@@ -4,5 +4,4 @@
   <xacro:macro name="color_sensor" params="prefix parent visualize:=false *origin1 **origin2">
     <xacro:property name="parent_link" value="${parent}"/>
-    <xacro:property name="color_sensor_len" value="0.05"/>
     <link name="${prefix}_color_sensor">
         <visual>

Commit message: Adressed requested changes
Improved readability, changed colors aproach, removed unused variables, cleaned includes

File: ca_description/urdf/sensors/color_sensor.xacro (robot description, xacro)
@@ -2,5 +2,5 @@
 <robot xmlns:xacro="http://ros.org/wiki/xacro">
   <xacro:include filename="$(find ca_description)/urdf/common_properties.xacro"/>
-  <xacro:macro name="color_sensor" params="name_prefix color parent visualize:=false *origin">
+  <xacro:macro name="color_sensor" params="name_prefix color parent *origin">
     <xacro:property name="parent_link" value="${parent}"/>
     <link name="${name_prefix}_color_sensor">
